File: Sync-chan.kicad_pcb (KiCad board)
At the start: 4 copper layers, 100 x 97 mm, 62 parts, among them J1 Jack-DC, J2 AudioJack3_Ring_Switch, J3 AudioJack3_Ring_Switch, J4 AudioJack3_Ring_Switch, J5 AudioJack3_Ring_Switch, J6 AudioJack3_Ring_Switch, SW1 SW_SPDT, U1 LM358MX, U2 TM1627_7seg_driver, U3 Arduino_Nano_v3.x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

Commit message: correct footprints
Parts:
- U2: footprint Sync-chan:TM1627_SOP28 -> Sync-chan:SOIC-28
Routing:
- net /S1: track 79.0 -> 80.7 mm
- net /S4: track 40.1 -> 41.6 mm
- net /S3: track 53.1 -> 54.2 mm
- net /S2: track 64.3 -> 65.2 mm
Other:
- board text added: "Sync-chan"
- board text added: "by Kinoshita Lab. 2020"

Commit message: modify pcb
Parts:
- U2: footprint Sync-chan:SOIC-28 -> Sync-chan:TM1627_SO
