File: Sync-chan.sch (KiCad schematic (older format))
At the start: 60 parts, among them J1 Jack-DC, J2 AudioJack3_Ring_Switch, J3 AudioJack3_Ring_Switch, J4 AudioJack3_Ring_Switch, J5 AudioJack3_Ring_Switch, J6 AudioJack3_Ring_Switch, SW1 SW_SPDT, U1 LM358MX, U2 TM1627_7seg_driver, U3 Arduino_Nano_v3.x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

Commit message: correct footprints
Parts:
- U2: footprint Sync-chan:TM1627_SOP28 -> Sync-chan:SOIC-28
Changed lines of the file:
@@
 F 0 "U2" H 12075 5715 50  0000 C CNN
 F 1 "TM1627_7seg_driver" H 12075 5624 50  0000 C CNN
-F 2 "Sync-chan:TM1627_SOP28" H 12100 3550 50  0001 C CNN
+F 2 "Sync-chan:SOIC-28" H 12100 3550 50  0001 C CNN
 F 3 "" H 12100 3550 50  0001 C CNN
 	1    12100 4700

Commit message: modify pcb
Parts:
- U2: footprint Sync-chan:SOIC-28 -> Sync-chan:TM1627_SO
Changed lines of the file:
@@
 F 0 "U2" H 12075 5715 50  0000 C CNN
 F 1 "TM1627_7seg_driver" H 12075 5624 50  0000 C CNN
-F 2 "Sync-chan:SOIC-28" H 12100 3550 50  0001 C CNN
+F 2 "Sync-chan:TM1627_SO" H 12100 3550 50  0001 C CNN
 F 3 "" H 12100 3550 50  0001 C CNN
 	1    12100 4700
