File: hardware/Sync-chan.sch (KiCad schematic (older format))
At the start: 60 parts, among them J1 Jack-DC, J2 AudioJack3_Ring_Switch, J3 AudioJack3_Ring_Switch, J4 AudioJack3_Ring_Switch, J5 AudioJack3_Ring_Switch, J6 AudioJack3_Ring_Switch, SW1 SW_SPDT, U1 LM358MX, U2 TM1627_7seg_driver, U3 Arduino_Nano_v3.x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

Commit message: move files
Parts:
- removed 7SEG-1, 7SEG-2, 7SEG-3, 7SEG-4, 7SEG-5: A-551SRD-A_7seg, Sync-chan:A-551SRD-A 7seg, symbol Sync-chan:A-551SRD-A_7seg
- removed C3, C4, C5: 100p, Capacitors_SMD:C_0603_HandSoldering, symbol Device:C
- removed R4, R5: 10k, Resistors_SMD:R_0603_HandSoldering, symbol Device:R
- removed U2: TM1627_7seg_driver, Sync-chan:TM1627_SO, symbol Sync-chan:TM1627_7seg_driver
- added 7SEG-1: 7seg_4digit_cathode_common_OSL40562-LR, Sync-chan:7seg_4digit_cathode_common_OSL40562-LR, symbol Sync-chan:7seg_4digit_cathode_common_OSL40562-LR
- added H5, H6: MountingHole, Mounting_Holes:MountingHole_3.2mm_M3, symbol Mechanical:MountingHole
- added U2: TM1640_7seg_driver, Housings_SOIC:SOIC-28W_7.5x18.7mm_Pitch1.27mm, symbol Sync-chan:TM1640_7seg_driver
- R2: value 1k -> 10k
Connections:
- net labels added: A, B, C, D, DIGIT1, DIGIT2, DIGIT3, DIGIT4, DIN, DP, E, F, G, SCLK
- net labels removed: CLK, DIO, G1, G2, G3, G4, G5, G6, G7, LED_Sync, S1, S2, S3, S4, S5, STB
- wire segments 153 -> 119
- no-connect marks 37 -> 39
Other:
- moved on the sheet: C6, C7, U3

Commit message: replace C1, C7, modify TRS symbol
Parts:
- C1, C7: footprint Capacitors_SMD:C_1206_HandSoldering -> Capacitor_SMD:CP_Elec_6.3x7.7; symbol Device:C -> Device:CP
Changed lines of the file:
@@
 $EndComp
 $Comp
-L Device:C C1
+L Device:CP C1
 U 1 1 5CDB5ED1
 P 3400 1450
 F 0 "C1" H 3515 1496 50  0000 L CNN
 F 1 "100u" H 3515 1405 50  0000 L CNN
-F 2 "Capacitors_SMD:C_1206_HandSoldering" H 3438 1300 50  0001 C CNN
+F 2 "Capacitor_SMD:CP_Elec_6.3x7.7" H 3438 1300 50  0001 C CNN
 F 3 "~" H 3400 1450 50  0001 C CNN
 	1    3400 1450
@@
 $EndComp
 $Comp
-L Device:C C7
+L Device:CP C7
 U 1 1 5E97DEBC
 P 5600 4400
 F 0 "C7" H 5715 4446 50  0000 L CNN
 F 1 "100u" H 5715 4355 50  0000 L CNN
-F 2 "Capacitors_SMD:C_1206_HandSoldering" H 5638 4250 50  0001 C CNN
+F 2 "Capacitor_SMD:CP_Elec_6.3x7.7" H 5638 4250 50  0001 C CNN
 F 3 "~" H 5600 4400 50  0001 C CNN
 	1    5600 4400
