File: hardware/Sync-chan.kicad_pcb (KiCad board)
At the start: 4 copper layers, 100 x 97 mm, 53 parts, among them J1 Jack-DC, J2 AudioJack3_Ring_Switch, J3 AudioJack3_Ring_Switch, J4 AudioJack3_Ring_Switch, J5 AudioJack3_Ring_Switch, J6 AudioJack3_Ring_Switch, SW1 SW_SPDT, U1 LM358MX, U2 TM1640_7seg_driver, U3 Arduino_Nano_v3.x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

Commit message: correct footprint molex trs connector
Routing:
- net Net-(J6-PadT): track 27.6 -> 19.1 mm
- net Net-(J3-PadT): track 64.5 -> 56.6 mm
- net Net-(J4-PadT): track 56.1 -> 48.2 mm
- net Net-(J5-PadT): track 41.3 -> 33.5 mm
- net Net-(J2-PadT): track 42.8 -> 44.4 mm

Commit message: replace C1, C7, modify TRS symbol
Parts:
- C1, C7: footprint Capacitors_SMD:C_1206_HandSoldering -> Capacitor_SMD:CP_Elec_6.3x7.7
- moved C1 5.09 mm to (139.2, 66.5), turned to 0 degrees
- moved C7 1.90 mm to (173.2, 92.0)
Connections:
- J2 pad R: (no net) -> Net-(J2-PadR)
- J2 pad TN: (no net) -> Net-(J2-PadTN)
- J3 pad R: (no net) -> Net-(J3-PadR)
- J3 pad TN: (no net) -> Net-(J3-PadTN)
- J4 pad R: (no net) -> Net-(J4-PadR)
- J4 pad TN: (no net) -> Net-(J4-PadTN)
- J5 pad R: (no net) -> Net-(J5-PadR)
- J5 pad TN: (no net) -> Net-(J5-PadTN)
- J6 pad R: (no net) -> Net-(J6-PadR)
- J6 pad TN: (no net) -> Net-(J6-PadTN)
- SW1 pad 3: (no net) -> Net-(SW1-Pad3)
- U2 pad 1: (no net) -> Net-(U2-Pad1)
- U2 pad 2: (no net) -> Net-(U2-Pad2)
- U2 pad 22: (no net) -> Net-(U2-Pad22)
- U2 pad 23: (no net) -> Net-(U2-Pad23)
- U2 pad 24: (no net) -> Net-(U2-Pad24)
- U2 pad 25: (no net) -> Net-(U2-Pad25)
- U2 pad 26: (no net) -> Net-(U2-Pad26)
- U2 pad 27: (no net) -> Net-(U2-Pad27)
- U2 pad 28: (no net) -> Net-(U2-Pad28)
- U2 pad 3: (no net) -> Net-(U2-Pad3)
- U2 pad 4: (no net) -> Net-(U2-Pad4)
- U3 pad 1: (no net) -> Net-(U3-Pad1)
- U3 pad 16: (no net) -> Net-(U3-Pad16)
- U3 pad 17: (no net) -> Net-(U3-Pad17)
- U3 pad 18: (no net) -> Net-(U3-Pad18)
- U3 pad 2: (no net) -> Net-(U3-Pad2)
- U3 pad 22: (no net) -> Net-(U3-Pad22)
- U3 pad 23: (no net) -> Net-(U3-Pad23)
- U3 pad 24: (no net) -> Net-(U3-Pad24)
- U3 pad 25: (no net) -> Net-(U3-Pad25)
- U3 pad 26: (no net) -> Net-(U3-Pad26)
- U3 pad 28: (no net) -> Net-(U3-Pad28)
- U3 pad 3: (no net) -> Net-(U3-Pad3)
- U3 pad 30: (no net) -> Net-(U3-Pad30)
- U3 pad 9: (no net) -> Net-(U3-Pad9)
- U4 pad 12: (no net) -> Net-(U4-Pad12)
- U4 pad 15: (no net) -> Net-(U4-Pad15)
Routing:
- net GND: track 85.9 -> 93.2 mm
